File: ecad/UPS/controller.kicad_sch (KiCad schematic)
At the start: 32 parts, among them J2 PROG, SW1 SW_Push, SW2 SW_Push, U1 STM32L152RCT6, U2 AP2112K-3.3TRG1

Commit message: Update controller.kicad_sch
Parts:
- renumbered COUT to C3, CIN to C4, decouplingcapateachVDDpin to C5, decouplingcapateachVDDpin1 to C6, decouplingcapateachVDDpin2 to C7, decouplingcapateachVDDpin3 to C8, decouplingcapateachVDDpin4 to C9, R4 to R1, pull-upresistors to R10, R1 to R11, R1 to R12, R2 to R13, R4 to R14, R5 to R2, R6 to R3, R7 to R4, otherpullups to R5, otherpullups1 to R6, otherpullups2 to R7, otherpullups3 to R8, pull-upresistoronSDA to R9
Changed lines of the file:
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@@
 		(on_board yes)
 		(dnp no)
-		(property "Reference" "pull-upresistors"
-			(at 27.432 117.602 0)
+		(property "Reference" "R10"
+			(at 38.354 117.856 0)
 			(effects
 				(font
@@
 			(project "controller"
 				(path "/50450634-21c9-467c-beaf-30f36150c371"
-					(reference "pull-upresistors")
+					(reference "R10")
 					(unit 1)
 				)
@@
 		(dnp no)
 		(fields_autoplaced yes)
-		(property "Reference" "decouplingcapateachVDDpin1"
+		(property "Reference" "C6"
 			(at 138.43 137.1599 0)
 			(effects
@@
 			(project "controller"
 				(path "/50450634-21c9-467c-beaf-30f36150c371"
-					(reference "decouplingcapateachVDDpin1")
+					(reference "C6")
 					(unit 1)
 				)
@@
 		(on_board yes)
 		(dnp no)
-		(property "Reference" "R5"
+		(property "Reference" "R2"
 			(at 227.1014 128.1684 0)
 			(effects
@@
 			(project "controller"
 				(path "/50450634-21c9-467c-beaf-30f36150c371"
-					(reference "R5")
+					(reference "R2")
 					(unit 1)
 				)
@@
 		(on_board yes)
 		(dnp no)
-		(property "Reference" "R2"
+		(property "Reference" "R13"
 			(at 86.2584 21.8186 0)
 			(effects
@@
 			(project "controller"
 				(path "/50450634-21c9-467c-beaf-30f36150c371"
-					(reference "R2")
+					(reference "R13")
 					(unit 1)
 				)
@@
 		(dnp no)
 		(fields_autoplaced yes)
-		(property "Reference" "decouplingcapateachVDDpin"
+		(property "Reference" "C5"
 			(at 144.78 137.1599 0)
 			(effects
@@
 			(project "controller"
 				(path "/50450634-21c9-467c-beaf-30f36150c371"
-					(reference "decouplingcapateachVDDpin")
+					(reference "C5")
 					(unit 1)
 				)
@@
 		(on_board yes)
 		(dnp no)
-		(property "Reference" "R1"
+		(property "Reference" "R11"
 			(at 86.2584 35.7886 0)
 			(effects
@@
 			(project "controller"
 				(path "/50450634-21c9-467c-beaf-30f36150c371"
-					(reference "R1")
+					(reference "R11")
 					(unit 1)
 				)
@@
 		(on_board yes)
 		(dnp no)
-		(property "Reference" "R1"
+		(property "Reference" "R12"
 			(at 86.2584 29.4386 0)
 			(effects
@@
 			(project "controller"
 				(path "/50450634-21c9-467c-beaf-30f36150c371"
-					(reference "R1")
+					(reference "R12")
 					(unit 1)
 				)
@@
 		(dnp no)
 		(fields_autoplaced yes)
-		(property "Reference" "R7"
+		(property "Reference" "R4"
 			(at 26.67 99.0599 0)
 			(effects
@@
 			(project "controller"
 				(path "/50450634-21c9-467c-beaf-30f36150c371"
-					(reference "R7")
+					(reference "R4")
 					(unit 1)
 				)
@@
 		(dnp no)
 		(fields_autoplaced yes)
-		(property "Reference" "otherpullups"
+		(property "Reference" "R5"
 			(at 76.2 118.1099 0)
 			(effects
@@
 			(project "controller"
 				(path "/50450634-21c9-467c-beaf-30f36150c371"
-					(reference "otherpullups")
+					(reference "R5")
 					(unit 1)
 				)
@@
 		(dnp no)
 		(fields_autoplaced yes)
-		(property "Reference" "otherpullups1"
+		(property "Reference" "R6"
 			(at 71.12 118.1099 0)
 			(effects
@@
 			(project "controller"
 				(path "/50450634-21c9-467c-beaf-30f36150c371"
-					(reference "otherpullups1")
+					(reference "R6")
 					(unit 1)
 				)
@@
 		(dnp no)
 		(fields_autoplaced yes)
-		(property "Reference" "pull-upresistoronSDA"
+		(property "Reference" "R9"
 			(at 52.07 118.1099 0)
 			(effects
@@
 			(project "controller"
 				(path "/50450634-21c9-467c-beaf-30f36150c371"
-					(reference "pull-upresistoronSDA")
+					(reference "R9")
 					(unit 1)
 				)
@@
 		(dnp no)
 		(fields_autoplaced yes)
-		(property "Reference" "decouplingcapateachVDDpin3"
+		(property "Reference" "C8"
 			(at 128.27 137.1599 0)
 			(effects
@@
 			(project "controller"
 				(path "/50450634-21c9-467c-beaf-30f36150c371"
-					(reference "decouplingcapateachVDDpin3")
+					(reference "C8")
 					(unit 1)
 				)
@@
 		(on_board yes)
 		(dnp no)
-		(property "Reference" "R4"
+		(property "Reference" "R1"
 			(at 189.0014 134.5184 0)
 			(effects
@@
 			(project "controller"
 				(path "/50450634-21c9-467c-beaf-30f36150c371"
-					(reference "R4")
+					(reference "R1")
 					(unit 1)
 				)
@@
 		(dnp no)
 		(fields_autoplaced yes)
-		(property "Reference" "COUT"
+		(property "Reference" "C3"
 			(at 97.79 158.7499 0)
 			(effects
@@
 			(project "controller"
 				(path "/50450634-21c9-467c-beaf-30f36150c371"
-					(reference "COUT")
+					(reference "C3")
 					(unit 1)
 				)
@@
 		(dnp no)
 		(fields_autoplaced yes)
-		(property "Reference" "R6"
+		(property "Reference" "R3"
 			(at 92.71 116.8399 0)
 			(effects
@@
 			(project ""
 				(path "/50450634-21c9-467c-beaf-30f36150c371"
-					(reference "R6")
+					(reference "R3")
 					(unit 1)
 				)
@@
 		(dnp no)
 		(fields_autoplaced yes)
-		(property "Reference" "otherpullups3"
+		(property "Reference" "R8"
 			(at 60.96 118.1099 0)
 			(effects
@@
 			(project "controller"
 				(path "/50450634-21c9-467c-beaf-30f36150c371"
-					(reference "otherpullups3")
+					(reference "R8")
 					(unit 1)
 				)
@@
 		(dnp no)
 		(fields_autoplaced yes)
-		(property "Reference" "CIN"
+		(property "Reference" "C4"
 			(at 52.07 156.2099 0)
 			(effects
@@
 			(project "controller"
 				(path "/50450634-21c9-467c-beaf-30f36150c371"
-					(reference "CIN")
+					(reference "C4")
 					(unit 1)
 				)
@@
 		(on_board yes)
 		(dnp no)
-		(property "Reference" "R4"
+		(property "Reference" "R14"
 			(at 86.2584 19.2786 0)
 			(effects
@@
 			(project "controller"
 				(path "/50450634-21c9-467c-beaf-30f36150c371"
-					(reference "R4")
+					(reference "R14")
 					(unit 1)
 				)
@@
 		(dnp no)
 		(fields_autoplaced yes)
-		(property "Reference" "decouplingcapateachVDDpin4"
+		(property "Reference" "C9"
 			(at 123.19 137.1599 0)
 			(effects
@@
 			(project "controller"
 				(path "/50450634-21c9-467c-beaf-30f36150c371"
-					(reference "decouplingcapateachVDDpin4")
+					(reference "C9")
 					(unit 1)
 				)
@@
 		(dnp no)
 		(fields_autoplaced yes)
-		(property "Reference" "otherpullups2"
+		(property "Reference" "R7"
 			(at 66.04 118.1099 0)
 			(effects
@@
 			(project "controller"
 				(path "/50450634-21c9-467c-beaf-30f36150c371"
-					(reference "otherpullups2")
+					(reference "R7")
 					(unit 1)
 				)
@@
 		(dnp no)
 		(fields_autoplaced yes)
-		(property "Reference" "decouplingcapateachVDDpin2"
+		(property "Reference" "C7"
 			(at 133.35 137.1599 0)
 			(effects
@@
 			(project "controller"
 				(path "/50450634-21c9-467c-beaf-30f36150c371"
-					(reference "decouplingcapateachVDDpin2")
+					(reference "C7")
 					(unit 1)
 				)

Commit message: Add thermistors for batteries and link signals
Connections:
- net bat_th1: now reaches U1.34 (PB13)
- net bat_th2: now reaches U1.35 (PB14)
- net bat_th3: now reaches U1.36 (PB15)
Changed lines of the file:
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@@
+	(wire
+		(pts
+			(xy 100.33 121.92) (xy 106.68 121.92)
+		)
+		(stroke
+			(width 0)
+			(type default)
+		)
+	)
 	(wire
 		(pts
@@
 	(wire
 		(pts
+			(xy 100.33 124.46) (xy 106.68 124.46)
+		)
+		(stroke
+			(width 0)
+			(type default)
+		)
+	)
+	(wire
+		(pts
 			(xy 234.95 119.38) (xy 234.95 120.65)
 		)
@@
 		(pts
 			(xy 130.81 132.08) (xy 130.81 133.35)
+		)
+		(stroke
+			(width 0)
+			(type default)
+		)
+	)
+	(wire
+		(pts
+			(xy 100.33 127) (xy 106.68 127)
 		)
 		(stroke
@@
 		)
 	)
+	(hierarchical_label "bat_th3"
+		(shape input)
+		(at 100.33 127 180)
+		(effects
+			(font
+				(size 1.27 1.27)
+			)
+			(justify right)
+		)
+	)
 	(hierarchical_label "CMPIN"
 		(shape input)
@@
 		)
 	)
+	(hierarchical_label "bat_th1"
+		(shape input)
+		(at 100.33 121.92 180)
+		(effects
+			(font
+				(size 1.27 1.27)
+			)
+			(justify right)
+		)
+	)
 	(hierarchical_label "cmp_out"
 		(shape input)
@@
 	)
 	(hierarchical_label "i2c_scl"
-		(shape input)
+		(shape bidirectional)
 		(at 39.37 104.14 180)
 		(effects
@@
 		)
 	)
+	(hierarchical_label "bat_th2"
+		(shape input)
+		(at 100.33 124.46 180)
+		(effects
+			(font
+				(size 1.27 1.27)
+			)
+			(justify right)
+		)
+	)
 	(hierarchical_label "i2c_sda"
-		(shape input)
+		(shape bidirectional)
 		(at 39.37 106.68 180)
 		(effects

Commit message: found a short
Connections:
- net GND: no longer D1.1 (K), R11.1
- new net: D1.1 (K), R11.1
Changed lines of the file:
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@@
-	)
-	(junction
-		(at 87.63 34.29)
-		(diameter 0)
-		(color 0 0 0 0)
 	)
 	(junction
@@
 	)
 	(junction
-		(at 82.55 34.29)
-		(diameter 0)
-		(color 0 0 0 0)
-	)
-	(junction
 		(at 124.46 142.24)
 		(diameter 0)
@@
 		)
 		(stroke
-			(width 0)
-			(type default)
-		)
-	)
-	(wire
-		(pts
-			(xy 82.55 34.29) (xy 87.63 34.29)
-		)
-		(stroke

Commit message: PCB Outline
Parts:
- renumbered C2 to C4, C1 to C61, C4 to CIN1, C3 to COUT1, D1 to D10, D1 to D6, D4 to D8, D2 to D9, R4 to R18, R3 to R19, R14 to R20, R13 to R21, R12 to R22, R1 to R23, R2 to R29, R11 to R33, SW2 to SW1, SW1 to SW2, U1 to U4, U2 to U5, C9 to decouplingcapateachVDDpin1, C8 to decouplingcapateachVDDpin2, C7 to decouplingcapateachVDDpin3, C6 to decouplingcapateachVDDpin4, C5 to decouplingcapateachVDDpin5, R8 to otherpullups1, R7 to otherpullups2, R6 to otherpullups3, R5 to otherpullups4, R9 to pull-upresistoronSDA1, R10 to pull-upresistors1
Connections:
- net 3.3V: now also COUT1.1, R19.2, U4.13 (VDDA), U4.19 (VDD_4), U4.32 (VDD_1), U4.48 (VDD_2), U4.64 (VDD_3), U5.5 (VOUT), decouplingcapateachVDDpin1.2, decouplingcapateachVDDpin2.2, decouplingcapateachVDDpin3.2, decouplingcapateachVDDpin4.2, decouplingcapateachVDDpin5.2, otherpullups1.2, otherpullups2.2, otherpullups3.2, otherpullups4.2, pull-upresistoronSDA1.1, pull-upresistors1.1
