File: ecad/UPS/BoostConvertor.kicad_sch (KiCad schematic)
At the start: 24 parts

Commit message: Introduce fuses and a bit more routing
Connections:
- net 5v renamed vbus
Changed lines of the file:
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@@
 		)
 	)
-	(hierarchical_label "5v"
-		(shape input)
+	(hierarchical_label "vbus"
+		(shape output)
 		(at 203.2 71.12 0)
 		(effects
