File: ecad/UPS/BoostConvertor.kicad_sch (KiCad schematic)
At the start: 24 parts

Commit message: Rename all grounds to GND
Parts:
- TP3: value PGNDTest -> GNDTest
Connections:
- net AGND is gone; now on net GND: C23.2, C35.2, C36.2, NT1.1, PS1.10 (AGND), R30.2, R31.2, TP2.1
- net PGND is gone; now on net GND: C18.2, C19.2, C21.2, C24.2, C25.2, C26.2, C3.2, NT1.2, PS1.3 (PGND), TP3.1
Changed lines of the file:
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@@
 		)
 	)
-	(global_label "AGND"
+	(global_label "GND"
 		(shape input)
 		(at 132.08 60.96 90)
@@
 		)
 	)
-	(global_label "PGND"
+	(global_label "GND"
 		(shape input)
 		(at 123.19 90.17 270)
@@
 		)
 	)
-	(global_label "AGND"
+	(global_label "GND"
 		(shape input)
 		(at 129.54 90.17 270)
@@
 		)
 	)
-	(global_label "AGND"
+	(global_label "GND"
 		(shape input)
 		(at 157.48 91.44 270)
@@
 		)
 		(property "Intersheetrefs" "${INTERSHEET_REFS}"
-			(at 157.48 99.3843 90)
+			(at 157.48 98.2957 90)
 			(hide yes)
 			(show_name no)
@@
 		)
 	)
-	(global_label "PGND"
+	(global_label "GND"
 		(shape input)
 		(at 63.5 66.04 270)
@@
 		)
 	)
-	(global_label "AGND"
+	(global_label "GND"
 		(shape input)
 		(at 137.16 97.79 270)
@@
 		)
 		(property "Intersheetrefs" "${INTERSHEET_REFS}"
-			(at 137.16 105.7343 90)
+			(at 137.16 104.6457 90)
 			(hide yes)
 			(show_name no)
@@
 		)
 	)
-	(global_label "AGND"
+	(global_label "GND"
 		(shape input)
 		(at 57.15 85.09 180)
@@
 		)
 	)
-	(global_label "PGND"
+	(global_label "GND"
 		(shape input)
 		(at 62.23 85.09 0)
@@
 		)
 	)
-	(global_label "PGND"
+	(global_label "GND"
 		(shape input)
 		(at 200.66 82.55 270)
@@
 		)
 		(property "Intersheetrefs" "${INTERSHEET_REFS}"
-			(at 200.66 90.6757 90)
+			(at 200.66 89.4057 90)
 			(hide yes)
 			(show_name no)
@@
 		)
 	)
-	(global_label "PGND"
+	(global_label "GND"
 		(shape input)
 		(at 78.74 80.01 270)
@@
 		)
 		(instances
+			(project "BoostConvertor"
+				(path "/88bd6fb1-4e06-4886-ab3d-9bc9521a3d03"
+					(reference "C20")
+					(unit 1)
+				)
+			)
 			(project "UPS"
 				(path "/9d92b60a-4a6b-449c-b462-cab19e69d38c/66173f08-558e-4192-bd35-ba55c00529e3"
@@
 		)
 		(instances
+			(project "BoostConvertor"
+				(path "/88bd6fb1-4e06-4886-ab3d-9bc9521a3d03"
+					(reference "C36")
+					(unit 1)
+				)
+			)
 			(project "UPS"
 				(path "/9d92b60a-4a6b-449c-b462-cab19e69d38c/66173f08-558e-4192-bd35-ba55c00529e3"
@@
 		)
 		(instances
+			(project "BoostConvertor"
+				(path "/88bd6fb1-4e06-4886-ab3d-9bc9521a3d03"
+					(reference "C35")
+					(unit 1)
+				)
+			)
 			(project "UPS"
 				(path "/9d92b60a-4a6b-449c-b462-cab19e69d38c/66173f08-558e-4192-bd35-ba55c00529e3"
@@
 		)
 		(instances
+			(project "BoostConvertor"
+				(path "/88bd6fb1-4e06-4886-ab3d-9bc9521a3d03"
+					(reference "R38")
+					(unit 1)
+				)
+			)
 			(project "UPS"
 				(path "/9d92b60a-4a6b-449c-b462-cab19e69d38c/66173f08-558e-4192-bd35-ba55c00529e3"
@@
 		)
 		(instances
+			(project "BoostConvertor"
+				(path "/88bd6fb1-4e06-4886-ab3d-9bc9521a3d03"
+					(reference "TP4")
+					(unit 1)
+				)
+			)
 			(project "UPS"
 				(path "/9d92b60a-4a6b-449c-b462-cab19e69d38c/66173f08-558e-4192-bd35-ba55c00529e3"
@@
 		)
 		(instances
+			(project "BoostConvertor"
+				(path "/88bd6fb1-4e06-4886-ab3d-9bc9521a3d03"
+					(reference "R30")
+					(unit 1)
+				)
+			)
 			(project "UPS"
 				(path "/9d92b60a-4a6b-449c-b462-cab19e69d38c/66173f08-558e-4192-bd35-ba55c00529e3"
@@
 		)
 		(instances
+			(project "BoostConvertor"
+				(path "/88bd6fb1-4e06-4886-ab3d-9bc9521a3d03"
+					(reference "C18")
+					(unit 1)
+				)
+			)
 			(project "UPS"
 				(path "/9d92b60a-4a6b-449c-b462-cab19e69d38c/66173f08-558e-4192-bd35-ba55c00529e3"
@@
 			)
 		)
-		(property "Value" "PGNDTest"
+		(property "Value" "GNDTest"
 			(at 205.74 82.5499 90)
 			(show_name no)
@@
 		)
 		(instances
+			(project "BoostConvertor"
+				(path "/88bd6fb1-4e06-4886-ab3d-9bc9521a3d03"
+					(reference "TP3")
+					(unit 1)
+				)
+			)
 			(project "UPS"
 				(path "/9d92b60a-4a6b-449c-b462-cab19e69d38c/66173f08-558e-4192-bd35-ba55c00529e3"
@@
 		)
 		(instances
+			(project "BoostConvertor"
+				(path "/88bd6fb1-4e06-4886-ab3d-9bc9521a3d03"
+					(reference "C24")
+					(unit 1)
+				)
+			)
 			(project "UPS"
 				(path "/9d92b60a-4a6b-449c-b462-cab19e69d38c/66173f08-558e-4192-bd35-ba55c00529e3"
@@
 		)
 		(instances
+			(project "BoostConvertor"
+				(path "/88bd6fb1-4e06-4886-ab3d-9bc9521a3d03"
+					(reference "NT1")
+					(unit 1)
+				)
+			)
 			(project "UPS"
 				(path "/9d92b60a-4a6b-449c-b462-cab19e69d38c/66173f08-558e-4192-bd35-ba55c00529e3"
@@
 		)
 		(instances
+			(project "BoostConvertor"
+				(path "/88bd6fb1-4e06-4886-ab3d-9bc9521a3d03"
+					(reference "C23")
+					(unit 1)
+				)
+			)
 			(project "UPS"
 				(path "/9d92b60a-4a6b-449c-b462-cab19e69d38c/66173f08-558e-4192-bd35-ba55c00529e3"
@@
 		)
 		(instances
+			(project "BoostConvertor"
+				(path "/88bd6fb1-4e06-4886-ab3d-9bc9521a3d03"
+					(reference "C26")
+					(unit 1)
+				)
+			)
 			(project "UPS"
 				(path "/9d92b60a-4a6b-449c-b462-cab19e69d38c/66173f08-558e-4192-bd35-ba55c00529e3"
@@
 		)
 		(instances
+			(project "BoostConvertor"
+				(path "/88bd6fb1-4e06-4886-ab3d-9bc9521a3d03"
+					(reference "C19")
+					(unit 1)
+				)
+			)
 			(project "UPS"
 				(path "/9d92b60a-4a6b-449c-b462-cab19e69d38c/66173f08-558e-4192-bd35-ba55c00529e3"
@@
 		)
 		(instances
+			(project "BoostConvertor"
+				(path "/88bd6fb1-4e06-4886-ab3d-9bc9521a3d03"
+					(reference "TP2")
+					(unit 1)
+				)
+			)
 			(project "UPS"
 				(path "/9d92b60a-4a6b-449c-b462-cab19e69d38c/66173f08-558e-4192-bd35-ba55c00529e3"
@@
 		)
 		(instances
+			(project "BoostConvertor"
+				(path "/88bd6fb1-4e06-4886-ab3d-9bc9521a3d03"
+					(reference "#PWR0105")
+					(unit 1)
+				)
+			)
 			(project "UPS"
 				(path "/9d92b60a-4a6b-449c-b462-cab19e69d38c/66173f08-558e-4192-bd35-ba55c00529e3"
@@
 		)
 		(instances
+			(project "BoostConvertor"
+				(path "/88bd6fb1-4e06-4886-ab3d-9bc9521a3d03"
+					(reference "C21")
+					(unit 1)
+				)
+			)
 			(project "UPS"
 				(path "/9d92b60a-4a6b-449c-b462-cab19e69d38c/66173f08-558e-4192-bd35-ba55c00529e3"
@@
 		)
 		(instances
+			(project "BoostConvertor"
+				(path "/88bd6fb1-4e06-4886-ab3d-9bc9521a3d03"
+					(reference "TP5")
+					(unit 1)
+				)
+			)
 			(project "UPS"
 				(path "/9d92b60a-4a6b-449c-b462-cab19e69d38c/66173f08-558e-4192-bd35-ba55c00529e3"
@@
 		)
 		(instances
+			(project "BoostConvertor"
+				(path "/88bd6fb1-4e06-4886-ab3d-9bc9521a3d03"
+					(reference "L2")
+					(unit 1)
+				)
+			)
 			(project "UPS"
 				(path "/9d92b60a-4a6b-449c-b462-cab19e69d38c/66173f08-558e-4192-bd35-ba55c00529e3"
@@
 		)
 		(instances
+			(project "BoostConvertor"
+				(path "/88bd6fb1-4e06-4886-ab3d-9bc9521a3d03"
+					(reference "C25")
+					(unit 1)
+				)
+			)
 			(project "UPS"
 				(path "/9d92b60a-4a6b-449c-b462-cab19e69d38c/66173f08-558e-4192-bd35-ba55c00529e3"
@@
 		)
 		(instances
+			(project "BoostConvertor"
+				(path "/88bd6fb1-4e06-4886-ab3d-9bc9521a3d03"
+					(reference "TP1")
+					(unit 1)
+				)
+			)
 			(project "UPS"
 				(path "/9d92b60a-4a6b-449c-b462-cab19e69d38c/66173f08-558e-4192-bd35-ba55c00529e3"
@@
 		)
 		(instances
+			(project "BoostConvertor"
+				(path "/88bd6fb1-4e06-4886-ab3d-9bc9521a3d03"
+					(reference "R32")
+					(unit 1)
+				)
+			)
 			(project "UPS"
 				(path "/9d92b60a-4a6b-449c-b462-cab19e69d38c/66173f08-558e-4192-bd35-ba55c00529e3"
@@
 		)
 		(instances
+			(project "BoostConvertor"
+				(path "/88bd6fb1-4e06-4886-ab3d-9bc9521a3d03"
+					(reference "PS1")
+					(unit 1)
+				)
+			)
 			(project "UPS"
 				(path "/9d92b60a-4a6b-449c-b462-cab19e69d38c/66173f08-558e-4192-bd35-ba55c00529e3"
@@
 		)
 		(instances
+			(project "BoostConvertor"
+				(path "/88bd6fb1-4e06-4886-ab3d-9bc9521a3d03"
+					(reference "C22")
+					(unit 1)
+				)
+			)
 			(project "UPS"
 				(path "/9d92b60a-4a6b-449c-b462-cab19e69d38c/66173f08-558e-4192-bd35-ba55c00529e3"
@@
 		)
 		(instances
+			(project "BoostConvertor"
+				(path "/88bd6fb1-4e06-4886-ab3d-9bc9521a3d03"
+					(reference "R31")
+					(unit 1)
+				)
+			)
 			(project "UPS"
 				(path "/9d92b60a-4a6b-449c-b462-cab19e69d38c/66173f08-558e-4192-bd35-ba55c00529e3"
@@
 		)
 		(instances
+			(project "BoostConvertor"
+				(path "/88bd6fb1-4e06-4886-ab3d-9bc9521a3d03"
+					(reference "C3")
+					(unit 1)
+				)
+			)
 			(project "UPS"
 				(path "/9d92b60a-4a6b-449c-b462-cab19e69d38c/66173f08-558e-4192-bd35-ba55c00529e3"
@@
 		)
 	)
+	(sheet_instances
+		(path "/"
+			(page "1")
+		)
+	)
+	(embedded_fonts no)
 )

Commit message: Light PCB work
Also removed NetTie
Parts:
- removed NT1: NetTie_3, NetTie:NetTie-4_THT_Pad1.0mm, symbol Device:NetTie_3
Changed lines of the file:
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@@
-	(global_label "GND"
-		(shape input)
-		(at 57.15 85.09 180)
-		(fields_autoplaced yes)
-		(effects
-			(font
-				(size 1.27 1.27)
-			)
-			(justify right)
-		)
-		(property "Intersheetrefs" "${INTERSHEET_REFS}"
-			(at 49.2057 85.09 0)
-			(hide yes)
-			(show_name no)
-			(do_not_autoplace no)
-			(effects
-				(font
-					(size 1.27 1.27)
-				)
-				(justify right)
-			)
-		)
-	)
-	(global_label "GND"
-		(shape input)
-		(at 62.23 85.09 0)
-		(fields_autoplaced yes)
-		(effects
-			(font
-				(size 1.27 1.27)
-			)
-			(justify left)
-		)
-		(property "Intersheetrefs" "${INTERSHEET_REFS}"
-			(at 70.3557 85.09 0)
-			(hide yes)
-			(show_name no)
-			(do_not_autoplace no)
-			(effects
-				(font
-					(size 1.27 1.27)
-				)
-				(justify left)
-			)
-		)
-	)
 	(global_label "GND"
 		(shape input)
@@
 	)
 	(symbol
-		(lib_id "Device:NetTie_3")
-		(at 59.69 85.09 0)
-		(unit 1)
-		(body_style 1)
-		(exclude_from_sim no)
-		(in_bom no)
-		(on_board yes)
-		(in_pos_files yes)
-		(dnp no)
-		(fields_autoplaced yes)
-		(property "Reference" "NT1"
-			(at 59.69 80.01 0)
-			(show_name no)
-			(do_not_autoplace no)
-			(effects
-				(font
-					(size 1.27 1.27)
-				)
-			)
-		)
-		(property "Value" "NetTie_3"
-			(at 59.69 82.55 0)
-			(show_name no)
-			(do_not_autoplace no)
-			(effects
-				(font
-					(size 1.27 1.27)
-				)
-			)
-		)
-		(property "Footprint" "NetTie:NetTie-4_THT_Pad1.0mm"
-			(at 59.69 85.09 0)
-			(hide yes)
-			(show_name no)
-			(do_not_autoplace no)
-			(effects
-				(font
-					(size 1.27 1.27)
-				)
-			)
-		)
-		(property "Datasheet" ""
-			(at 59.69 85.09 0)
-			(hide yes)
-			(show_name no)
-			(do_not_autoplace no)
-			(effects
-				(font
-					(size 1.27 1.27)
-				)
-			)
-		)
-		(property "Description" "Net tie, 3 pins"
-			(at 59.69 85.09 0)
-			(hide yes)
-			(show_name no)
-			(do_not_autoplace no)
-			(effects
-				(font
-					(size 1.27 1.27)
-				)
-			)
-		)
-		(pin "2"
-		)
-		(pin "3"
-		)
-		(pin "1"
-		)
-		(instances
-			(project "BoostConvertor"
-				(path "/88bd6fb1-4e06-4886-ab3d-9bc9521a3d03"
-					(reference "NT1")
-					(unit 1)
-				)
-			)
-			(project "UPS"
-				(path "/9d92b60a-4a6b-449c-b462-cab19e69d38c/66173f08-558e-4192-bd35-ba55c00529e3"
-					(reference "NT1")
-					(unit 1)
-				)
-			)
-		)
-	)
-	(symbol
 		(lib_id "Device:C")
 		(at 146.05 86.36 0)
@@
 	)
 	(symbol
-		(lib_id "power:GND")
-		(at 57.15 87.63 0)
-		(unit 1)
-		(body_style 1)
-		(exclude_from_sim no)
-		(in_bom yes)
-		(on_board yes)
-		(in_pos_files yes)
-		(dnp no)
-		(fields_autoplaced yes)
-		(property "Reference" "#PWR0105"
-			(at 57.15 93.98 0)
-			(hide yes)
-			(show_name no)
-			(do_not_autoplace no)
-			(effects
-				(font
-					(size 1.27 1.27)
-				)
-			)
-		)
-		(property "Value" "GND"
-			(at 57.15 92.71 0)
-			(show_name no)
-			(do_not_autoplace no)
-			(effects
-				(font
-					(size 1.27 1.27)
-				)
-			)
-		)
-		(property "Footprint" ""
-			(at 57.15 87.63 0)
-			(hide yes)
-			(show_name no)
-			(do_not_autoplace no)
-			(effects
-				(font
-					(size 1.27 1.27)
-				)
-			)
-		)
-		(property "Datasheet" ""
-			(at 57.15 87.63 0)
-			(hide yes)
-			(show_name no)
-			(do_not_autoplace no)
-			(effects
-				(font
-					(size 1.27 1.27)
-				)
-			)
-		)
-		(property "Description" "Power symbol creates a global label with name \"GND\" , ground"
-			(at 57.15 87.63 0)
-			(hide yes)
-			(show_name no)
-			(do_not_autoplace no)
-			(effects
-				(font
-					(size 1.27 1.27)
-				)
-			)
-		)
-		(pin "1"
-		)
-		(instances
-			(project "BoostConvertor"
-				(path "/88bd6fb1-4e06-4886-ab3d-9bc9521a3d03"
-					(reference "#PWR0105")
-					(unit 1)
-				)
-			)
-			(project "UPS"
-				(path "/9d92b60a-4a6b-449c-b462-cab19e69d38c/66173f08-558e-4192-bd35-ba55c00529e3"
-					(reference "#PWR0105")
-					(unit 1)
-				)
-			)
-		)
-	)
-	(symbol
 		(lib_id "Device:C")
 		(at 78.74 76.2 0)
@@
 		)
 	)
-	(embedded_fonts no)
 )
