File: ecad/UPS/Charger.kicad_sch (KiCad schematic)
At the start: 68 parts, among them J1 Barrel_Jack, J2 Conn_01x02_Socket, Q1 CSD18540Q5B, Q2 Q_PMOS_DGS, Q4 Q_PMOS_DGS, Q5 CSD18540Q5B, Q6 CSD18540Q5B, Q7 CSD18540Q5B, U1 BQ25730RSNR

Commit message: Thermistor changes
Parts:
- removed J2: Conn_01x02_Socket, Connector_AMASS:AMASS_XT60-F_1x02_P7.20mm_Vertical, symbol Connector:Conn_01x02_Socket
- removed TH2, TH3, TH4: B57471V2104J062, Resistor_SMD:R_0805_2012Metric_Pad1.20x1.40mm_HandSolder, symbol Device:Thermistor_NTC
- added C68, C69, C70: 100 nF, Capacitor_SMD:C_0603_1608Metric, symbol Device:C
- added J2, J5, J6: Conn_01x02_Pin, symbol Connector:Conn_01x02_Pin
Connections:
- net GNDA: now also C68.2, C69.2, C70.2, J2.2 (Pin_2), J5.2 (Pin_2), J6.2 (Pin_2)
- net bat_th1: now also C70.1, J2.1 (Pin_1)
- net bat_th2: now also C69.1, J5.1 (Pin_1)
- net bat_th3: now also C68.1, J6.1 (Pin_1)
