File: ecad/UPS/UPS.kicad_pcb (KiCad board)
At the start: 4 copper layers, 121.9 x 139.7 mm, 163 parts, among them J2 Conn_01x02_Pin, J3 USB_C_Receptacle_USB2.0_16P, J4 PROG, J5 Conn_01x02_Pin, J6 Conn_01x02_Pin, J7 Fan_Connector, J8 PJ-002AH, Q1 CSD18540Q5B, Q2 Q_PMOS_DGS, Q3 IRLR7843TRPBF, Q4 Q_PMOS_DGS, Q5 CSD18540Q5B, Q6 CSD18540Q5B, Q7 CSD18540Q5B, Q8 2N7002, SW3 SW_DPDT_x2, U1 BQ25730RSNR, U2 MPQ5031GRE-0001-AEC1-P, U4 STM32L152RCT6, U5 AP2112K-3.3TRG1, U6 BOOT0, U7 NRST

Commit message: Most of the second switching stage done
Parts:
- moved Q3 82.8 mm to (163.0, 141.8), turned to 0 degrees
- moved J3 72.0 mm to (167.5, 114.5), turned to 90 degrees
- moved D5 63.1 mm to (158.3, 115.0), turned to -90 degrees
- moved SW3 59.1 mm to (142.5, 145.5), turned to 0 degrees
- moved R8 43.6 mm to (157.5, 79.5), turned to -90 degrees
- moved U2 30.9 mm to (126.0, 139.5)
- moved R5 27.0 mm to (133.0, 53.5), turned to 0 degrees
- moved CIN1 21.9 mm to (151.5, 81.5)
- moved R1 17.4 mm to (121.0, 64.0)
- moved C53 14.2 mm to (149.2, 43.5), turned to 0 degrees
- moved C52 14.2 mm to (149.2, 57.6), turned to 0 degrees
- moved C51 9.95 mm to (149.2, 55.5), turned to 0 degrees
- moved R13 9.25 mm to (127.5, 68.0), turned to 180 degrees
- moved C54 9.17 mm to (149.2, 46.0), turned to 0 degrees
- moved C38 8.08 mm to (132.0, 63.5)
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Routing:
- net VDDA: track 0.00 -> 33.0 mm, vias 0 -> 3
- net Net-(U1-LODRV2): track 0.00 -> 25.4 mm, vias 0 -> 2
- net Net-(U1-HIDRV2): track 0.00 -> 21.9 mm, vias 0 -> 2
- net REGN: track 0.00 -> 12.3 mm
- net BTST2: track 0.00 -> 8.87 mm
- net Net-(U1-IADPT): track 0.00 -> 8.21 mm, vias 0 -> 2
- net GND: track 20.3 -> 27.8 mm
- net Net-(U1-SW2): track 0.00 -> 1.86 mm
- added copper zone on F.Cu, net Net-(U1-SW2)
